Commit message: UR5e에 Robotiq 2F-85 그리퍼 결합 및 컨트롤 슬라이더 추가

File: public/models/ur5e/ur5e_web.urdf (robot description, URDF)
Before this commit: robot ur5e, 13 links, 12 joints
Links:
- added link robotiq_85_base_link; visual mesh filename=gripper/visual/robotiq_base.dae
- added link robotiq_85_left_finger_link; visual mesh filename=gripper/visual/left_finger.dae
- added link robotiq_85_left_finger_tip_link; visual mesh filename=gripper/visual/left_finger_tip.dae
- added link robotiq_85_left_inner_knuckle_link; visual mesh filename=gripper/visual/left_inner_knuckle.dae
- added link robotiq_85_left_knuckle_link; visual mesh filename=gripper/visual/left_knuckle.dae
- added link robotiq_85_right_finger_link; visual mesh filename=gripper/visual/right_finger.dae
- added link robotiq_85_right_finger_tip_link; visual mesh filename=gripper/visual/right_finger_tip.dae
- added link robotiq_85_right_inner_knuckle_link; visual mesh filename=gripper/visual/right_inner_knuckle.dae
- added link robotiq_85_right_knuckle_link; visual mesh filename=gripper/visual/right_knuckle.dae
Joints:
- added joint gripper_base_joint: type fixed, parent tool0, child robotiq_85_base_link, origin xyz=0 0 0 rpy=0 0 0
- added joint robotiq_85_left_finger_joint: type fixed, parent robotiq_85_left_knuckle_link, child robotiq_85_left_finger_link, origin xyz=0.03152616 0.0 -0.00376347 rpy=0 0 0
- added joint robotiq_85_left_finger_tip_joint: type revolute, parent robotiq_85_left_finger_link, child robotiq_85_left_finger_tip_link, origin xyz=0.00563134 0.0 0.04718515 rpy=0 0 0, axis 0 -1 0, limit lower=-0.8 upper=0.0 effort=50 velocity=0.5, mimic joint=robotiq_85_left_knuckle_joint multiplier=-1
- added joint robotiq_85_left_inner_knuckle_joint: type revolute, parent robotiq_85_base_link, child robotiq_85_left_inner_knuckle_link, origin xyz=0.0127 0.0 0.06142 rpy=0 0 0, axis 0 -1 0, limit lower=0.0 upper=0.8 effort=50 velocity=0.5, mimic joint=robotiq_85_left_knuckle_joint
- added joint robotiq_85_left_knuckle_joint: type revolute, parent robotiq_85_base_link, child robotiq_85_left_knuckle_link, origin xyz=0.03060114 0.0 0.05490452 rpy=0 0 0, axis 0 -1 0, limit lower=0.0 upper=0.8 effort=50 velocity=0.5
- added joint robotiq_85_right_finger_joint: type fixed, parent robotiq_85_right_knuckle_link, child robotiq_85_right_finger_link, origin xyz=-0.03152616 0.0 -0.00376347 rpy=0 0 0
- added joint robotiq_85_right_finger_tip_joint: type revolute, parent robotiq_85_right_finger_link, child robotiq_85_right_finger_tip_link, origin xyz=-0.00563134 0.0 0.04718515 rpy=0 0 0, axis 0 -1 0, limit lower=0.0 upper=0.8 effort=50 velocity=0.5, mimic joint=robotiq_85_left_knuckle_joint
- added joint robotiq_85_right_inner_knuckle_joint: type revolute, parent robotiq_85_base_link, child robotiq_85_right_inner_knuckle_link, origin xyz=-0.0127 0.0 0.06142 rpy=0 0 0, axis 0 -1 0, limit lower=-0.8 upper=0.0 effort=50 velocity=0.5, mimic joint=robotiq_85_left_knuckle_joint multiplier=-1
- added joint robotiq_85_right_knuckle_joint: type revolute, parent robotiq_85_base_link, child robotiq_85_right_knuckle_link, origin xyz=-0.03060114 0.0 0.05490452 rpy=0 0 0, axis 0 -1 0, limit lower=-0.8 upper=0.0 effort=50 velocity=0.5, mimic joint=robotiq_85_left_knuckle_joint multiplier=-1
